File: main/main.sch (KiCad schematic (older format))
At the start: 18 parts, among them J1 USB_C_Receptacle, Q1 BSS138, SW1 SW_SPST, SW2 SW_SPST, SW3 SW_SPST, SW4 SW_SPST, SW5 SW_SPST, SW6 SW_SPST, U1 LN6206P332MR-G

Commit message: made spacer layer, replaces Ws2813 with WS2812, fixed fabrication for v0.0.0, now v0.1.0
Parts:
- removed J1: USB_C_Receptacle, william_usb:C168688, symbol Connector:USB_C_Receptacle
- added J1: USB_C_Receptacle_USB2.0, william_usb:C168688, symbol Connector:USB_C_Receptacle_USB2.0
- C4: value 10U -> 4U7
- U1: symbol william_dc_ldo:LN6206P332MR-G -> main-rescue:LN6206P332MR-G-william_dc_ldo
Connections:
- net +5V: now also J1.A4 (VBUS), J1.A9 (VBUS), J1.B4 (VBUS), J1.B9 (VBUS)
- net GND: now also J1.A1 (GND), J1.A12 (GND), J1.B1 (GND), J1.B12 (GND), J1.S1 (SHIELD)
Changed lines of the file:
@@
 EESchema Schematic File Version 4
+LIBS:main-cache
 EELAYER 30 0
 EELAYER END
@@
 U 5DEECD42
 F0 "LEDs" 50
-F1 "led_array.sch" 50
+F1 "2812_mini_led_array.sch" 50
 F2 "5V" I L 10000 3700 50
 F3 "DIN" I L 10000 3850 50
@@
 P 6250 1350
 F 0 "C4" H 6365 1396 50  0000 L CNN
-F 1 "10U" H 6365 1305 50  0000 L CNN
+F 1 "4U7" H 6365 1305 50  0000 L CNN
 F 2 "Capacitor_SMD:C_0402_1005Metric" H 6288 1200 50  0001 C CNN
 F 3 "~" H 6250 1350 50  0001 C CNN
@@
 Wire Wire Line
 	4500 1500 5350 1500
-Text Notes 5850 1700 0    50   ~ 0
+Text Notes 5250 900  0    50   ~ 0
 LCSC pn:\nC141407
 $Comp
-L william_dc_ldo:LN6206P332MR-G U1
+L main-rescue:LN6206P332MR-G-william_dc_ldo U1
 U 1 1 5DF1CFB8
 P 5350 1250
@@
 Text Label 9500 3850 1    50   ~ 0
 ~LED_DATA_OUT~_5V
-$Comp
-L Connector:USB_C_Receptacle J1
-U 1 1 5E1B7ADE
-P 1100 1850
-F 0 "J1" H 1207 3117 50  0000 C CNN
-F 1 "USB_C_Receptacle" H 1207 3026 50  0000 C CNN
-F 2 "william_usb:C168688" H 1250 1850 50  0001 C CNN
-F 3 "https://www.usb.org/sites/default/files/documents/usb_type-c.zip" H 1250 1850 50  0001 C CNN
-	1    1100 1850
-	1    0    0    -1
-$EndComp
 Text Label 6100 4150 0    50   ~ 0
 LED_DATA_OUT_3V3
@@
 	7600 4050 8400 4050
 Wire Wire Line
-	1100 3500 1100 3450
-Connection ~ 1100 3500
-Wire Wire Line
-	800  3500 1100 3500
-Wire Wire Line
-	800  3450 800  3500
-Wire Wire Line
-	1100 3550 1100 3500
+	1100 2400 1100 2350
+Connection ~ 1100 2400
+Wire Wire Line
+	800  2400 1100 2400
+Wire Wire Line
+	800  2350 800  2400
+Wire Wire Line
+	1100 2450 1100 2400
 $Comp
 L power:GND #PWR04
 U 1 1 5F9ED8FF
-P 1100 3550
-F 0 "#PWR04" H 1100 3300 50  0001 C CNN
-F 1 "GND" H 1105 3377 50  0000 C CNN
-F 2 "" H 1100 3550 50  0001 C CNN
-F 3 "" H 1100 3550 50  0001 C CNN
-	1    1100 3550
+P 1100 2450
+F 0 "#PWR04" H 1100 2200 50  0001 C CNN
+F 1 "GND" H 1105 2277 50  0000 C CNN
+F 2 "" H 1100 2450 50  0001 C CNN
+F 3 "" H 1100 2450 50  0001 C CNN
+	1    1100 2450
 	1    0    0    -1
 $EndComp
@@
 L power:PWR_FLAG #FLG0102
 U 1 1 5E220D8A
-P 1400 3500
-F 0 "#FLG0102" H 1400 3575 50  0001 C CNN
-F 1 "PWR_FLAG" H 1400 3673 50  0000 C CNN
-F 2 "" H 1400 3500 50  0001 C CNN
-F 3 "~" H 1400 3500 50  0001 C CNN
-	1    1400 3500
-	1    0    0    -1
-$EndComp
-Wire Wire Line
-	1400 3500 1100 3500
+P 1400 2400
+F 0 "#FLG0102" H 1400 2475 50  0001 C CNN
+F 1 "PWR_FLAG" H 1400 2573 50  0000 C CNN
+F 2 "" H 1400 2400 50  0001 C CNN
+F 3 "~" H 1400 2400 50  0001 C CNN
+	1    1400 2400
+	1    0    0    -1
+$EndComp
+Wire Wire Line
+	1400 2400 1100 2400
 Wire Wire Line
 	2050 850  1800 850
 Connection ~ 1800 850
+$Comp
+L Connector:USB_C_Receptacle_USB2.0 J1
+U 1 1 5DF2CF3E
+P 1100 1450
+F 0 "J1" H 1207 2317 50  0000 C CNN
+F 1 "USB_C_Receptacle_USB2.0" H 1207 2226 50  0000 C CNN
+F 2 "william_usb:C168688" H 1250 1450 50  0001 C CNN
+F 3 "https://www.usb.org/sites/default/files/documents/usb_type-c.zip" H 1250 1450 50  0001 C CNN
+	1    1100 1450
+	1    0    0    -1
+$EndComp
 $EndSCHEMATC
